File: hardware/project-mute-button.kicad_pcb (KiCad board)
At the start: 2 copper layers, 72.8 x 35.4 mm, 16 parts, among them J1 Conn_01x06_Female, J2 Conn_01x06_Female, J3 Button, J4 Toggle Switch, Q1 Q_NMOS_GSD

Commit message: Routing done
Parts:
- moved J3 32.0 mm to (83.3, 66.3)
- moved J4 32.0 mm to (51.4, 66.3)
Routing:
- net +5V: track 0.00 -> 63.1 mm
- net +3V3: track 0.00 -> 51.0 mm
- net /G0: track 0.00 -> 30.9 mm
- net /G2: track 0.00 -> 24.6 mm
- net /G1: track 0.00 -> 14.9 mm
- net GND: track 0.00 -> 11.1 mm, vias 0 -> 5
- net Net-(D2-Pad2): track 0.00 -> 4.53 mm
- net Net-(D1-Pad2): track 0.00 -> 4.53 mm
- net Net-(D1-Pad1): track 65.1 -> 66.5 mm
- added copper zone on B.Cu, net GND
Changed lines of the file:
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@@
     (thickness 1.6)
     (drawings 34)
-    (tracks 6)
+    (tracks 65)
     (zones 0)
     (modules 16)
@@
   )
   (setup
-    (last_trace_width 0.5)
+    (last_trace_width 1)
     (user_trace_width 0.5)
+    (user_trace_width 1)
     (trace_clearance 0.2)
     (zone_clearance 0.508)
@@
   )
   (module TZ022101B000G:TZ022101B000G (layer F.Cu)
-    (at 83.35 66.35 180)
+    (at 51.35 66.35 180)
     (fp_text reference J4 (at 0 5.85) (layer F.SilkS) hide
       (effects (font (size 1 1) (thickness 0.15)))
@@
   )
   (module TZ022101B000G:TZ022101B000G (layer F.Cu)
-    (at 51.35 66.35 180)
+    (at 83.35 66.35 180)
     (fp_text reference J3 (at 0 5.85) (layer F.SilkS) hide
       (effects (font (size 1 1) (thickness 0.15)))
@@
   (gr_line (start 41.75 24.75) (end 67.35 24.75) (layer Dwgs.User) (width 0.15))
   (gr_line (start 41.75 95.55) (end 67.35 95.55) (layer Edge.Cuts) (width 0.05))
-  (segment (start 92.6375 63.85) (end 97.35 68.5625) (width 0.5) (layer F.Cu) (net 14))
-  (segment (start 68.35 65.35) (end 69.85 63.85) (width 0.5) (layer F.Cu) (net 14))
-  (segment (start 69.85 63.85) (end 92.6375 63.85) (width 0.5) (layer F.Cu) (net 14))
-  (segment (start 66.85 63.85) (end 68.35 65.35) (width 0.5) (layer F.Cu) (net 14))
-  (segment (start 37.35 68.5625) (end 42.0625 63.85) (width 0.5) (layer F.Cu) (net 14))
-  (segment (start 42.0625 63.85) (end 66.85 63.85) (width 0.5) (layer F.Cu) (net 14))
+  (segment (start 61.35 69.525) (end 63.35 69.525) (width 0.25) (layer F.Cu) (net 2))
+  (segment (start 79.175 69.525) (end 81.475001 67.224999) (width 0.25) (layer F.Cu) (net 2))
+  (segment (start 63.35 69.525) (end 79.175 69.525) (width 0.25) (layer F.Cu) (net 2))
+  (segment (start 85.224999 67.224999) (end 86.55 68.55) (width 0.25) (layer F.Cu) (net 2))
+  (segment (start 81.475001 67.224999) (end 85.224999 67.224999) (width 0.25) (layer F.Cu) (net 2))
+  (segment (start 78.13 83.27) (end 72.05 83.27) (width 0.25) (layer F.Cu) (net 2))
+  (segment (start 86.55 68.55) (end 86.55 74.85) (width 0.25) (layer F.Cu) (net 2))
+  (segment (start 86.55 74.85) (end 78.13 83.27) (width 0.25) (layer F.Cu) (net 2))
+  (segment (start 70.849999 87.149999) (end 72.05 88.35) (width 1) (layer F.Cu) (net 3))
+  (segment (start 55.439997 87.149999) (end 70.849999 87.149999) (width 1) (layer F.Cu) (net 3))
+  (segment (start 42.175 73.885002) (end 55.439997 87.149999) (width 1) (layer F.Cu) (net 3))
+  (segment (start 42.175 73.35) (end 42.175 73.885002) (width 1) (layer F.Cu) (net 3))
+  (segment (start 77.525 88.35) (end 72.05 88.35) (width 1) (layer F.Cu) (net 3))
+  (segment (start 92.525 73.35) (end 77.525 88.35) (width 1) (layer F.Cu) (net 3))
+  (via (at 73.75 85.85) (size 0.8) (drill 0.4) (layers F.Cu B.Cu) (net 6))
+  (segment (start 75.35 85.81) (end 73.79 85.81) (width 0.5) (layer F.Cu) (net 6))
+  (segment (start 73.79 85.81) (end 73.75 85.85) (width 0.5) (layer F.Cu) (net 6))
+  (segment (start 49.6 71.3) (end 49.6 68.5) (width 0.5) (layer F.Cu) (net 6))
+  (via (at 50.15 67.95) (size 0.8) (drill 0.4) (layers F.Cu B.Cu) (net 6))
+  (segment (start 49.6 68.5) (end 50.15 67.95) (width 0.5) (layer F.Cu) (net 6))
+  (via (at 82.05 67.95) (size 0.8) (drill 0.4) (layers F.Cu B.Cu) (net 6))
+  (segment (start 81.6 71.3) (end 81.6 68.4) (width 0.5) (layer F.Cu) (net 6))
+  (segment (start 81.6 68.4) (end 82.05 67.95) (width 0.5) (layer F.Cu) (net 6))
+  (segment (start 68.175 67.85) (end 68.85 67.85) (width 0.5) (layer F.Cu) (net 6))
+  (via (at 69.25 67.45) (size 0.8) (drill 0.4) (layers F.Cu B.Cu) (net 6))
+  (segment (start 68.85 67.85) (end 69.25 67.45) (width 0.5) (layer F.Cu) (net 6))
+  (via (at 65.25 66.05) (size 0.8) (drill 0.4) (layers F.Cu B.Cu) (net 6))
+  (segment (start 66.35 66) (end 65.3 66) (width 0.5) (layer F.Cu) (net 6))
+  (segment (start 65.3 66) (end 65.25 66.05) (width 0.5) (layer F.Cu) (net 6))
+  (segment (start 59.35 73.175) (end 61.35 71.175) (width 0.25) (layer F.Cu) (net 7))
+  (segment (start 59.35 78.19) (end 59.35 73.175) (width 0.25) (layer F.Cu) (net 7))
+  (segment (start 57.475 71.3) (end 59.35 73.175) (width 0.25) (layer F.Cu) (net 7))
+  (segment (start 53.1 71.3) (end 57.475 71.3) (width 0.25) (layer F.Cu) (net 7))
+  (segment (start 63.35 74.95) (end 62.65 75.65) (width 0.25) (layer F.Cu) (net 10))
+  (segment (start 63.35 71.175) (end 63.35 74.95) (width 0.25) (layer F.Cu) (net 10))
+  (segment (start 66.725 74.55) (end 63.35 71.175) (width 0.25) (layer F.Cu) (net 10))
+  (segment (start 84.65 74.55) (end 66.725 74.55) (width 0.25) (layer F.Cu) (net 10))
+  (segment (start 85.1 71.3) (end 85.1 74.1) (width 0.25) (layer F.Cu) (net 10))
+  (segment (start 85.1 74.1) (end 84.65 74.55) (width 0.25) (layer F.Cu) (net 10))
+  (segment (start 67.25 67.125) (end 66.525 67.85) (width 0.25) (layer F.Cu) (net 11))
+  (segment (start 66.35 64.7) (end 67.25 65.6) (width 0.25) (layer F.Cu) (net 11))
+  (segment (start 67.25 65.6) (end 67.25 67.125) (width 0.25) (layer F.Cu) (net 11))
+  (segment (start 61.15 79.23) (end 62.65 80.73) (width 0.25) (layer F.Cu) (net 11))
+  (segment (start 61.15 74.55) (end 61.15 79.23) (width 0.25) (layer F.Cu) (net 11))
+  (segment (start 62.25 73.45) (end 61.15 74.55) (width 0.25) (layer F.Cu) (net 11))
+  (segment (start 62.25 70.75) (end 62.25 73.45) (width 0.25) (layer F.Cu) (net 11))
+  (segment (start 61.55 67.85) (end 60.45 68.95) (width 0.25) (layer F.Cu) (net 11))
+  (segment (start 66.525 67.85) (end 61.55 67.85) (width 0.25) (layer F.Cu) (net 11))
+  (segment (start 60.45 68.95) (end 60.45 70.05) (width 0.25) (layer F.Cu) (net 11))
+  (segment (start 60.45 70.05) (end 60.75 70.35) (width 0.25) (layer F.Cu) (net 11))
+  (segment (start 60.75 70.35) (end 61.85 70.35) (width 0.25) (layer F.Cu) (net 11))
+  (segment (start 61.85 70.35) (end 62.25 70.75) (width 0.25) (layer F.Cu) (net 11))
+  (segment (start 37.35 70.175) (end 40.525 73.35) (width 1) (layer F.Cu) (net 13))
+  (segment (start 37.35 70.1375) (end 37.35 70.175) (width 1) (layer F.Cu) (net 13))
+  (segment (start 68.35 64.125) (end 68.35 65.35) (width 1) (layer F.Cu) (net 14))
+  (segment (start 37.35 68.5625) (end 42.7625 63.15) (width 1) (layer F.Cu) (net 14))
+  (segment (start 67.375 63.15) (end 68.35 64.125) (width 1) (layer F.Cu) (net 14))
+  (segment (start 42.7625 63.15) (end 67.375 63.15) (width 1) (layer F.Cu) (net 14))
+  (segment (start 89.425 64.125) (end 68.35 64.125) (width 1) (layer F.Cu) (net 14))
+  (segment (start 95.710328 65.65) (end 90.95 65.65) (width 1) (layer F.Cu) (net 14))
+  (segment (start 90.95 65.65) (end 89.425 64.125) (width 1) (layer F.Cu) (net 14))
+  (segment (start 97.35 68.5625) (end 97.35 67.289672) (width 1) (layer F.Cu) (net 14))
+  (segment (start 97.35 67.289672) (end 95.710328 65.65) (width 1) (layer F.Cu) (net 14))
+  (segment (start 94.175 73.3125) (end 97.35 70.1375) (width 1) (layer F.Cu) (net 15))
+  (segment (start 94.175 73.35) (end 94.175 73.3125) (width 1) (layer F.Cu) (net 15))
+  (zone (net 6) (net_name GND) (layer B.Cu) (hatch edge 0.508)
+    (connect_pads (clearance 0.508))
+    (min_thickness 0.254)
+    (fill yes (arc_segments 32) (thermal_gap 0.508) (thermal_bridge_width 0.508))
+    (polygon
+      (pts
+        (xy 103.75 95.55) (xy 30.95 95.55) (xy 30.95 24.75) (xy 103.75 24.75)
+      )
+    )
+  )
 )

Commit message: Add version silk
Other:
- board text added: "François Gervais 6 novembre 2022 v1.0.0"
Changed lines of the file:
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@@
   (general
     (thickness 1.6)
-    (drawings 34)
+    (drawings 35)
     (tracks 65)
     (zones 0)
@@
     )
   )
+  (gr_text "François Gervais\n6 novembre 2022\nv1.0.0" (at 78.65 78.75) (layer F.SilkS)
+    (effects (font (size 1 1) (thickness 0.15)) (justify left))
+  )
   (gr_arc (start 38.35 60.15) (end 33.85 60.15) (angle -180) (layer Edge.Cuts) (width 0.05))
