File: hardware/project-mute-button.kicad_pcb (KiCad board)
At the start: 2 copper layers, 72.8 x 35.4 mm, 14 parts, among them J1 Conn_01x06_Female, J2 Conn_01x06_Female, J3 Button, J4 Toggle Switch, Q1 Q_NMOS_GSD

Commit message: Add case drawing
Other:
- board text added: "1.3mm between PCB and case all around"
